Commit message: update dobot case

File: dobot/urdf/robot1.urdf (robot description, URDF)
Before this commit: robot dobot, 11 links, 10 joints
Links:
- added link base; visual mesh filename=package://dobot/urdf/meshes/base.stl scale=0.001 0.001 0.001
Joints:
- added joint base_fix: type fixed, parent base, child base_link, origin xyz=0 0 0.04 rpy=0 0 0
- joint black_pallet_fix: origin xyz=-0.3 0.2 0 rpy=0 0 0 -> xyz=-0.29 0.15 0 rpy=0 0 0; parent base_link -> base
- joint pallet_fix: origin xyz=-0.25 0.0 0 rpy=0 0 0 -> xyz=-0.25 -0.03 0 rpy=0 0 0; parent base_link -> base
